File: hardware/ltm-main/ltm-main.kicad_sch (KiCad schematic)
At the start: 34 parts, among them J1 BATERAI (dari BMS), J2 MOTOR KIRI, J3 MOTOR KANAN, J4 OLED 1.3in I2C, J5 KE PCB SENSOR, Q1 S8050, SW1 ON/OFF, SW2 A (MENU), SW3 B (OK), U1 ESP32 DevKit 30P CH340, U2 TB6612FNG, U3 MP1584 (5,0 V)

Commit message: Layout PCB v1-draft: PCB utama + PCB sensor, routing FreeRouting, DRC bersih
- J5 jadi lubang tembus untuk pin header J1 PCB sensor (celah antar papan 2,4 mm)
- Pola net class Power memakai awalan / untuk net berlabel
- gen_pcb.py: outline dari model mekanik v11, penempatan, routing, pour GND, DRC
- Render atas/bawah dan rakitan di hardware/render

Co-Authored-By: Claude Opus 5.5 <noreply@anthropic.com>
Claude-Session: https://claude.ai/code/session_016j7fGnGXJh3ke3RU3C9DKW
Parts:
- J5: footprint Connector_PinSocket_2.54mm:PinSocket_2x05_P2.54mm_Vertical -> Connector_PinHeader_2.54mm:PinHeader_2x05_P2.54mm_Vertical; now left out of the parts list
Other:
- note added: "6. KE PCB SENSOR (J5 = lubang tembus)"
- note added: "J5 tidak dipasang komponen: pin header J1 PCB sensor masuk dari bawah lewat lubang J5, disolder di atas"
- note removed: "6. KE PCB SENSOR (J5 di sisi bawah)"
Changed lines of the file:
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@@
     (stroke (width 0) (type dash))
   )
-  (text "6. KE PCB SENSOR (J5 di sisi bawah)" (at 224.79 146.685 0)
+  (text "6. KE PCB SENSOR (J5 = lubang tembus)" (at 224.79 146.685 0)
     (effects (font (size 2 2) (thickness 0.4) bold) (justify left bottom))
   )
+  (text "J5 tidak dipasang komponen: pin header J1 PCB sensor\nmasuk dari bawah lewat lubang J5, disolder di atas" (at 228.6 222.25 0)
+    (effects (font (size 1.27 1.27)) (justify left bottom))
+  )
   (symbol (lib_id "Connector_Generic:Conn_02x05_Odd_Even") (at 264.16 185.42 0) (unit 1)
-    (in_bom yes) (on_board yes) (dnp no)
+    (in_bom no) (on_board yes) (dnp no)
     (property "Reference" "J5" (at 265.43 177.8 0)
       (effects (font (size 1.27 1.27)))
@@
       (effects (font (size 1.27 1.27)))
     )
-    (property "Footprint" "Connector_PinSocket_2.54mm:PinSocket_2x05_P2.54mm_Vertical" (at 264.16 185.42 0)
+    (property "Footprint" "Connector_PinHeader_2.54mm:PinHeader_2x05_P2.54mm_Vertical" (at 264.16 185.42 0)
       (effects (font (size 1.27 1.27)) hide)
     )

Commit message: PCB utama v2: lebih sederhana dan gampang diakses untuk edukasi
- Skematik 34 -> 25 komponen: C2-C6 dan R5-R8 dibuang (modul sudah punya
  kapasitor, encoder pakai INPUT_PULLUP), D1 SS14 -> 1N5819 (semua THT).
- ESP32 keluar dari bawah dudukan baterai, ESP32/TB6612/OLED di socket,
  MP1584 + D1 + R1/R2 di bawah dudukan baterai, J1/SW1 di tepi kanan.
- OLED header di depan: layar tidak perlu diputar (U8G2_R0).
- Silkscreen kotak blok (DAYA, OTAK, DRIVER MOTOR, LAYAR, SUARA) + peta
  ALUR DAYA. DRC 0/0, 294 segmen, 9 via.
- Model 3D v12 ikut PCB utama v2; tepi dudukan baterai ke Y 29,5.

Co-Authored-By: Claude Opus 5.5 <noreply@anthropic.com>
Claude-Session: https://claude.ai/code/session_016j7fGnGXJh3ke3RU3C9DKW
Parts:
- removed C2, C4, C5, C6: 100nF, Capacitor_THT:C_Disc_D5.0mm_W2.5mm_P5.00mm, symbol Device:C
- removed C3: 10uF/16V, Capacitor_THT:CP_Radial_D5.0mm_P2.00mm, symbol Device:C_Polarized
- removed R5, R6, R7, R8: 10k, Resistor_THT:R_Axial_DIN0207_L6.3mm_D2.5mm_P7.62mm_Horizontal, symbol Device:R
- D1: value SS14 -> 1N5819; footprint Diode_SMD:D_SMA -> Diode_THT:D_DO-41_SOD81_P10.16mm_Horizontal
Other:
- note added: "Encoder: pakai pull-up internal ESP32 (INPUT_PULLUP)"
- note added: "Kapasitor kecil tidak dipasang: modul TB6612, MP1584, dan ESP32 sudah punya kapasitor sendiri"
- note removed: "R5-R8 pull-up encoder: boleh tidak dipasang bila encoder sudah punya pull-up"

Commit message: Sensor 16 titik + mux + LED, kabel pita, aturan cetak 0,8 mm
- PCB sensor v2: batang lurus 110 x 51 mm, 16x ITR20001 (jarak 6,5 mm),
  modul mux CD74HC4067, MCP23017 + 16 LED indikator, box header IDC J1
- PCB utama: J5 jadi box header IDC 2x6 (kabel pita ke PCB sensor),
  pin ESP32 disusun ulang supaya jalur tidak saling silang
- Aturan tempat cetak: jalur >= 0,8 mm (daya 1,2), clearance 0,5,
  via 1,6/0,8; kedua PCB 0 jalur putus, DRC bersih
- Charter/RAB: 16 sensor, total Rp896.000
- Model 3D v12: PCB sensor batang di dudukan 3D print + kabel pita,
  STEP dan render diperbarui

Co-Authored-By: Claude Opus 5.5 <noreply@anthropic.com>
Claude-Session: https://claude.ai/code/session_016j7fGnGXJh3ke3RU3C9DKW
Parts:
- removed H5, H6: M3, MountingHole:MountingHole_3.2mm_M3, symbol Mechanical:MountingHole
- removed J5: KE PCB SENSOR, Connector_PinHeader_2.54mm:PinHeader_2x05_P2.54mm_Vertical, symbol Connector_Generic:Conn_02x05_Odd_Even
- added J5: KE PCB SENSOR, Connector_IDC:IDC-Header_2x06_P2.54mm_Vertical, symbol Connector_Generic:Conn_02x06_Odd_Even
- added R5, R6: 10k, Resistor_THT:R_Axial_DIN0207_L6.3mm_D2.5mm_P7.62mm_Horizontal, symbol Device:R
- Q1: footprint Package_TO_SOT_THT:TO-92_Inline -> Package_TO_SOT_THT:TO-92_Inline_Wide
Connections:
- net S2 is gone; now on net VBAT_SENSE: U1.3 (GPIO39/VN)
- net S3 is gone; now on net BTN_A: U1.4 (GPIO34)
- net S4 is gone; now on net BTN_B: U1.5 (GPIO35)
- net +3V3: now also J5.6 (Pin_6), R5.1, R6.1
- net +5V: now also J5.2 (Pin_2)
- net AIN1: now also U1.23 (GPIO5); no longer U1.9 (GPIO26)
- net AIN2: now also U1.24 (GPIO17/TX2); no longer U1.10 (GPIO27)
- net BIN1: now also U1.26 (GPIO4); no longer U1.25 (GPIO16/RX2)
- net BIN2: now also U1.28 (GPIO15); no longer U1.24 (GPIO17/TX2)
- net BTN_A: now also R5.2; no longer U1.28 (GPIO15)
- net BTN_B: now also R6.2; no longer U1.27 (GPIO2)
- net ENC_L_A: now also U1.13 (GPIO13); no longer U1.22 (GPIO18)
- net ENC_L_B: now also U1.11 (GPIO14); no longer U1.21 (GPIO19)
- net ENC_R_B: now also U1.21 (GPIO19); no longer U1.23 (GPIO5)
- net GND: now also J5.4 (Pin_4), J5.8 (Pin_8)
- net IR_EN: now also U1.10 (GPIO27), J5.1 (Pin_1); no longer U1.13 (GPIO13)
- net PWMA: now also U1.22 (GPIO18); no longer U1.8 (GPIO25)
- net PWMB: now also U1.25 (GPIO16/RX2); no longer U1.11 (GPIO14)
- net SCL: now also J5.12 (Pin_12)
- net SDA: now also J5.10 (Pin_10)
- net STBY: now also U1.27 (GPIO2); no longer U1.26 (GPIO4)
- net VBAT_SENSE: no longer U1.7 (GPIO33)
- net S1 renamed SIG
- net SIG: now also J5.3 (Pin_3)
- net S5 renamed MUX_S3
- net MUX_S3: now also J5.11 (Pin_11)
- new net MUX_S0: J5.5 (Pin_5), U1.9 (GPIO26)
- new net MUX_S1: J5.7 (Pin_7), U1.8 (GPIO25)
- new net MUX_S2: J5.9 (Pin_9), U1.7 (GPIO33)
Other:
- note added: "6. KE PCB SENSOR (kabel pita IDC 12 pin)"
- note added: "GPIO34/35 tanpa pull-up internal: R5, R6"
- note added: "H1-H2 rangka, H3-H4 bahu + dudukan PCB sensor"
- note added: "Mux: SIG GPIO36, S0-S3 GPIO32/33/2/15 LED sensor: MCP23017 di bus I2C (0x20)"
- note added: "Pembaca baterai: 8,4 V -> 2,08 V ke GPIO39"
- note removed: "6. KE PCB SENSOR (J5 = lubang tembus)"
- note removed: "H1-H2 rangka, H3-H4 bahu, H5-H6 spacer PCB sensor"
- note removed: "J5 tidak dipasang komponen: pin header J1 PCB sensor masuk dari bawah lewat lubang J5, disolder di atas"
- note removed: "Pembaca baterai: 8,4 V -> 2,08 V ke GPIO33"
- note removed: "Pull-up internal ESP32 (INPUT_PULLUP)"
