File: hardware/ltm-sensor/ltm-sensor.kicad_sch (KiCad schematic)
At the start: 22 parts, among them J1 KE PCB UTAMA, Q1 AO3400, U1 ITR20001 (S1), U2 ITR20001 (S2), U3 ITR20001 (S3), U4 ITR20001 (S4), U5 ITR20001 (S5)

Commit message: Sensor 16 titik + mux + LED, kabel pita, aturan cetak 0,8 mm
- PCB sensor v2: batang lurus 110 x 51 mm, 16x ITR20001 (jarak 6,5 mm),
  modul mux CD74HC4067, MCP23017 + 16 LED indikator, box header IDC J1
- PCB utama: J5 jadi box header IDC 2x6 (kabel pita ke PCB sensor),
  pin ESP32 disusun ulang supaya jalur tidak saling silang
- Aturan tempat cetak: jalur >= 0,8 mm (daya 1,2), clearance 0,5,
  via 1,6/0,8; kedua PCB 0 jalur putus, DRC bersih
- Charter/RAB: 16 sensor, total Rp896.000
- Model 3D v12: PCB sensor batang di dudukan 3D print + kabel pita,
  STEP dan render diperbarui

Co-Authored-By: Claude Opus 5.5 <noreply@anthropic.com>
Claude-Session: https://claude.ai/code/session_016j7fGnGXJh3ke3RU3C9DKW
Parts:
- removed J1: KE PCB UTAMA, Connector_PinHeader_2.54mm:PinHeader_2x05_P2.54mm_Vertical, symbol Connector_Generic:Conn_02x05_Odd_Even
- added C2: 100nF, Capacitor_SMD:C_0805_2012Metric_Pad1.18x1.45mm_HandSolder, symbol Device:C
- added D1, D10, D11, D12, D13, D14, D15, D16, D2, D3, D4, D5, D6, D7, D8, D9: LED, LED_SMD:LED_0805_2012Metric_Pad1.15x1.40mm_HandSolder, symbol Device:LED
- added J1: KABEL PITA 12 PIN, Connector_IDC:IDC-Header_2x06_P2.54mm_Vertical, symbol Connector_Generic:Conn_02x06_Odd_Even
- added R13, R14, R15, R16, R17, R18, R19, R20, R21, R22, R23, R24, R42: 10k, Resistor_SMD:R_0805_2012Metric_Pad1.20x1.40mm_HandSolder, symbol Device:R
- added R25, R26, R27, R28, R29, R30, R31, R32, R33, R34, R35, R36, R37, R38, R39, R40: 330, Resistor_SMD:R_0805_2012Metric_Pad1.20x1.40mm_HandSolder, symbol Device:R
- added R41: 100, Resistor_SMD:R_0805_2012Metric_Pad1.20x1.40mm_HandSolder, symbol Device:R
- added U10: ITR20001 (S10), ltm:ITR20001, symbol ltm:ITR20001
- added U11: ITR20001 (S11), ltm:ITR20001, symbol ltm:ITR20001
- added U12: ITR20001 (S12), ltm:ITR20001, symbol ltm:ITR20001
- added U13: ITR20001 (S13), ltm:ITR20001, symbol ltm:ITR20001
- added U14: ITR20001 (S14), ltm:ITR20001, symbol ltm:ITR20001
- added U15: ITR20001 (S15), ltm:ITR20001, symbol ltm:ITR20001
- added U16: ITR20001 (S16), ltm:ITR20001, symbol ltm:ITR20001
- added U17: Modul CD74HC4067, ltm:CD74HC4067_Module, symbol ltm:CD74HC4067_Module
- added U18: MCP23017, Package_DIP:DIP-28_W7.62mm_Socket, symbol Interface_Expansion:MCP23017_SP
- added U6: ITR20001 (S6), ltm:ITR20001, symbol ltm:ITR20001
- added U7: ITR20001 (S7), ltm:ITR20001, symbol ltm:ITR20001
- added U8: ITR20001 (S8), ltm:ITR20001, symbol ltm:ITR20001
- added U9: ITR20001 (S9), ltm:ITR20001, symbol ltm:ITR20001
- R1, R2, R3, R4, R5: value 180 -> 120
- R11: value 100 -> 10k
- R6, R7, R8: value 10k -> 120
Connections:
- net +3V3: now also R11.1, R12.1, C2.1, J1.6 (Pin_6), R13.1, R14.1, R15.1, R16.1, R17.1, R18.1, R19.1, R20.1, R21.1, R22.1, R23.1, R24.1, U17.23 (VCC), U18.18 (~{RESET}), U18.9 (VDD); no longer R6.1, R7.1, R8.1
- net +5V: now also R6.1, R7.1, R8.1, J1.2 (Pin_2)
- net GND: now also C2.2, D1.1 (K), D10.1 (K), D11.1 (K), D12.1 (K), D13.1 (K), D14.1 (K), D15.1 (K), D16.1 (K), D2.1 (K), D3.1 (K), D4.1 (K), D5.1 (K), D6.1 (K), D7.1 (K), D8.1 (K), D9.1 (K), J1.4 (Pin_4), J1.8 (Pin_8), R42.2, U10.4 (E), U11.4 (E), U12.4 (E), U13.4 (E), U14.4 (E), U15.4 (E), U16.4 (E), U17.22 (EN), U17.24 (GND), U18.10 (VSS), U18.15 (A0), U18.16 (A1), U18.17 (A2), U6.4 (E), U7.4 (E), U8.4 (E), U9.4 (E); no longer R12.2
- net IR_EN: now also J1.1 (Pin_1), R41.1; no longer R11.1
- net IR_G: now also R41.2, R42.1; no longer R11.2, R12.1
- net LED_K: now also U10.2 (K), U12.2 (K), U14.2 (K), U16.2 (K), U6.2 (K), U8.2 (K); no longer U1.2 (K), U3.2 (K), U5.2 (K)
- net S1: now also R9.2, U17.1 (C0); no longer R6.2
- net S2: now also R10.2, U17.2 (C1); no longer R7.2
- net S3: now also R11.2, U17.3 (C2); no longer R8.2
- net S4: now also R12.2, U17.4 (C3); no longer R9.2
- net S5: now also R13.2, U17.5 (C4); no longer R10.2
- net LED_A1 renamed IR_A1
- net LED_A2 renamed IR_A2
- net IR_A2: now also U3.1 (A); no longer U2.1 (A)
- net LED_A3 renamed IR_A3
- net IR_A3: now also U5.1 (A); no longer U3.1 (A)
- net LED_A4 renamed IR_A4
- net IR_A4: now also U7.1 (A); no longer U4.1 (A)
- net LED_A5 renamed IR_A5
- net IR_A5: now also U9.1 (A); no longer U5.1 (A)
- new net IR_A6: R6.2, U11.1 (A)
- new net IR_A7: R7.2, U13.1 (A)
- new net IR_A8: R8.2, U15.1 (A)
- new net IR_M1: U1.2 (K), U2.1 (A)
- new net IR_M2: U3.2 (K), U4.1 (A)
- new net IR_M3: U5.2 (K), U6.1 (A)
- new net IR_M4: U7.2 (K), U8.1 (A)
- new net IR_M5: U10.1 (A), U9.2 (K)
- new net IR_M6: U11.2 (K), U12.1 (A)
- new net IR_M7: U13.2 (K), U14.1 (A)
- new net IR_M8: U15.2 (K), U16.1 (A)
- new net LD1: R25.1, U18.28 (GPA7)
- new net LD10: R34.1, U18.7 (GPB6)
- new net LD11: R35.1, U18.6 (GPB5)
- new net LD12: R36.1, U18.5 (GPB4)
- new net LD13: R37.1, U18.4 (GPB3)
- new net LD14: R38.1, U18.3 (GPB2)
- new net LD15: R39.1, U18.2 (GPB1)
- new net LD16: R40.1, U18.1 (GPB0)
- new net LD2: R26.1, U18.27 (GPA6)
- new net LD3: R27.1, U18.26 (GPA5)
- new net LD4: R28.1, U18.25 (GPA4)
- new net LD5: R29.1, U18.24 (GPA3)
- new net LD6: R30.1, U18.23 (GPA2)
- new net LD7: R31.1, U18.22 (GPA1)
- new net LD8: R32.1, U18.21 (GPA0)
- new net LD9: R33.1, U18.8 (GPB7)
- new net LDA1: D1.2 (A), R25.2
- new net LDA10: D10.2 (A), R34.2
- new net LDA11: D11.2 (A), R35.2
- new net LDA12: D12.2 (A), R36.2
- new net LDA13: D13.2 (A), R37.2
- new net LDA14: D14.2 (A), R38.2
- new net LDA15: D15.2 (A), R39.2
- new net LDA16: D16.2 (A), R40.2
- new net LDA2: D2.2 (A), R26.2
- new net LDA3: D3.2 (A), R27.2
- new net LDA4: D4.2 (A), R28.2
- new net LDA5: D5.2 (A), R29.2
- new net LDA6: D6.2 (A), R30.2
- new net LDA7: D7.2 (A), R31.2
- new net LDA8: D8.2 (A), R32.2
- new net LDA9: D9.2 (A), R33.2
- new net MUX_S0: J1.5 (Pin_5), U17.21 (S0)
- new net MUX_S1: J1.7 (Pin_7), U17.20 (S1)
- new net MUX_S2: J1.9 (Pin_9), U17.19 (S2)
- new net MUX_S3: J1.11 (Pin_11), U17.18 (S3)
- new net S10: R18.2, U10.3 (C), U17.10 (C9)
- new net S11: R19.2, U11.3 (C), U17.11 (C10)
- new net S12: R20.2, U12.3 (C), U17.12 (C11)
- new net S13: R21.2, U13.3 (C), U17.13 (C12)
- new net S14: R22.2, U14.3 (C), U17.14 (C13)
- new net S15: R23.2, U15.3 (C), U17.15 (C14)
- new net S16: R24.2, U16.3 (C), U17.16 (C15)
- new net S6: R14.2, U17.6 (C5), U6.3 (C)
- new net S7: R15.2, U17.7 (C6), U7.3 (C)
- new net S8: R16.2, U17.8 (C7), U8.3 (C)
- new net S9: R17.2, U17.9 (C8), U9.3 (C)
- new net SCL: J1.12 (Pin_12), U18.12 (SCK)
- new net SDA: J1.10 (Pin_10), U18.13 (SDA)
- new net SIG: J1.3 (Pin_3), U17.17 (SIG)
- no-connect marks 0 -> 4
Other:
- note added: "2. SENSOR GARIS S1-S16 (ITR20001), LED IR dipasang seri berdua"
- note added: "3. SAKLAR LED IR"
- note added: "4. MULTIPLEXER 16 KE 1 (modul CD74HC4067)"
- note added: "5. LED INDIKATOR TIAP SENSOR (MCP23017, I2C alamat 0x20)"
- note added: "H1-H2: baut ke dudukan 3D print"
- note added: "Kabel pita IDC 2x6 ke J5 PCB utama"
- note added: "Kanal C0-C15 = S1-S16 (C0 = S1). Modul dicolok di socket female"
- note added: "LED IR: (5 V - 2 x 1,2 V) / 120 = +-21 mA per pasang, total +-170 mA lewat Q1"
- note added: "LED1-8 = GPA7..GPA0, LED9-16 = GPB7..GPB0. MCP sumber arus: (3,3 - 1,9) / 330 = +-4 mA"
- note removed: "2. SENSOR GARIS S1-S5 (ITR20001)"
- note removed: "3. SAKLAR LED IR (emitter ON/OFF)"
- note removed: "4. LUBANG BAUT M3"
- note removed: "IR_EN HIGH = LED menyala (baca ON - OFF)"
- note removed: "LED IR: (5 V - 1,2 V) / 180 = 21 mA per sensor, total +-105 mA lewat Q1"
- title: LTM - PCB Sensor Jangkar -> LTM - PCB Sensor 16 titik
